File: KiCad/LDAD_ABS_ENCLOSURE_52X48_1.69_LCD_TFT_16_bit_INA237.kicad_pcb (KiCad board)
At the start: 2 copper layers, 52.9 x 46.4 mm, 110 parts, among them CN3065_C2 4.7uF, CN3065_R1 1K8, CN3065_STDBY_LED1 LED, CN3965_C1 22uF, J1 TYPE-C-31-M-12, U1 MCP1525-TT, U2 ATSHA204A-MAHDA-T, U3 Battery_charger_CN3065_QFN8, U4 AHT20, U5 INA237AIDGSR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

Commit message: Add files via upload
Parts:
- removed the ? at (210.9, 77.7)
- removed the ? at (215.5, 77.7)
- removed ExtSW1: Conn_01x03_Female, Connector_JST:JST_SH_SM03B-SRSS-TB_1x03-1MP_P1.00mm_Horizontal
- removed the REF** at (210.6, 78.6)
- removed the REF** at (215.2, 78.6)
- added REF**: TestPoint_Keystone_5005-5009_Compact, TestPoint:TestPoint_Keystone_5005-5009_Compact, F.Cu at (217.9, 75.7)
- added REF**: TestPoint_Keystone_5005-5009_Compact, TestPoint:TestPoint_Keystone_5005-5009_Compact, F.Cu at (210.2, 75.7)
- moved TP2 39.1 mm to (209.3, 112.7)
- moved TP1 39.0 mm to (216.5, 112.5)
- moved TP3 38.5 mm to (212.7, 112.5)
- moved ER1 8.13 mm to (214.1, 77.8)
- moved I2C_SDA_R1 6.79 mm to (224.2, 81.2), turned to 180 degrees
- moved ATH20_C2 6.72 mm to (221.6, 82.0)
- moved I2C_SCL_R1 6.64 mm to (224.2, 82.9)
- moved MTRR1 4.69 mm to (204.1, 93.4)
- moved INA4_C1 4.57 mm to (206.2, 85.8), turned to 90 degrees
- moved MTRT1 4.16 mm to (207.1, 93.1)
- moved IMR2 2.45 mm to (209.3, 86.0)
- moved PWR_FUSE1 1.41 mm to (204.4, 101.9)
- moved AUR_C1 0.99 mm to (200.8, 102.6)
- moved U4 0.87 mm to (223.2, 76.5)
- moved IC_ENS1 0.87 mm to (230.6, 77.4)
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Connections:
- ESP32S1 pad 38: TEMT6000_IO33 -> INA237_ALRT_IO33
- ESP32S1 pad 39: PLUG_PWR_3V3_EN_IO38 -> unconnected-(ESP32S1-GPIO34-Pad39)
- ESP32S1 pad 40: unconnected-(ESP32S1-GPIO35-Pad40) -> TEMT6000_IO35
- TMPR1 pad 2: TEMT6000_IO33 -> TEMT6000_IO35
- U5 pad 3: INA237_ALRT_IO -> INA237_ALRT_IO33
- U6 pad EMITTER: TEMT6000_IO33 -> TEMT6000_IO35
Routing:
- net TEMT6000_IO35: track 0.00 -> 92.2 mm, vias 0 -> 3
- net TEMT6000_IO33: track 91.4 -> 0.00 mm, vias 3 -> 0
- net VIN: track 86.5 -> 53.3 mm, vias 3 -> 4
- net ADC_VOUT: track 29.6 -> 0.00 mm, vias 3 -> 0
- net INA237_ALRT_IO33: track 0.00 -> 28.7 mm, vias 0 -> 2
- net GPIO9_I2C_SCL: track 100.9 -> 77.6 mm, vias 6 -> 5
- net GPIO8_I2C_SDA: track 102.6 -> 80.1 mm
- net 3V3: track 260.3 -> 281.9 mm, vias 18 -> 20
- net INA237_PROBE_+: track 0.00 -> 18.4 mm
- net INA237_PROBE_-: track 0.00 -> 13.0 mm
- net GNDD: track 162.3 -> 168.0 mm
- net ADC_A0: track 5.23 -> 0.00 mm, vias 1 -> 0
- net USB_D+: track 43.6 -> 47.7 mm
- net USB_D-: track 46.4 -> 50.4 mm
- net USB_5V0F: track 32.6 -> 35.6 mm
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- added copper zone on F.Cu, net INA237_PROBE_+
- added copper zone on F.Cu, net INA237_PROBE_-
Other:
- board text added: "16-Bit Power Measurements"
- board text added: "IN"
- board text added: "MAX 85V"
- board text added: "OUT"
- board text added: "PCB rev. 11-2023"
- board text added: "VOLTAGE HIGH"
- board text removed: "0R"
- board text removed: "16-Bit DAQ"
- board text removed: "1K"
- board text removed: "200K"
- board text removed: "20K"
- board text removed: "2M"
- board text removed: "ADC"
- board text removed: "DAC IN"
- board text removed: "DAC Vout"
- board text removed: "Ohmmeter selection"
- board text removed: "PCB rev. 10-2023"
- board text removed: "PUL"
