File: KiCad/LDAD_ABS_ENCLOSURE_52X48_1.69_LCD_TFT_16_bit_INA237.kicad_sch (KiCad schematic)
At the start: 83 parts, among them CN3065_C2 4.7uF, CN3065_R1 1K8, CN3065_STDBY_LED1 LED, CN3965_C1 22uF, J1 Conn_01x07_Socket, J1 TYPE-C-31-M-12, J3 U.FL-R-SMT(01), J6 RFShield_OnePiece, U1 ATSHA204A-MAHDA-T, U1 MCP1525-TT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

Commit message: Add files via upload
Parts:
- removed ExtSW1: Conn_01x03_Female, Connector_JST:JST_SH_SM03B-SRSS-TB_1x03-1MP_P1.00mm_Horizontal, symbol Connector:Conn_01x03_Female
Connections:
- net TEMT6000_IO35: now reaches ESP32S1.40 (GPIO35)
- net TEMT6000_IO35: now also TMPR1.2, U6.EMITTER
- net INA237_ALRT_IO renamed INA237_ALRT_IO33
- net INA237_ALRT_IO33: now also ESP32S1.38 (GPIO33)
- net PLUG_PWR_3V3_EN_IO38: no longer names the net of ESP32S1.39 (GPIO34)
- removed net TEMT6000_IO33: ESP32S1.38 (GPIO33), TMPR1.2, U6.EMITTER
